File: osw-light.kicad_pcb (KiCad board)
At the start: 4 copper layers, 36.1 x 36.1 mm, 56 parts, among them J1 Conn_02x12_Odd_Even, J2 Conn_01x06, Q1 2N7002, U1 RV-3028-C7, U2 LIS2DTW12TR, U3 ESP32-PICO-D4, U4 XC6209, U5 BQ51050BRHL, U6 XC6209

Commit message: Added dormant file from my local git
Other:
- rule pad_to_mask_clearance: 0.0508 -> 0
Changed lines of the file:
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@@
       (dielectric_constraints no)
     )
-    (pad_to_mask_clearance 0.0508)
-    (pad_to_paste_clearance 0.1016)
+    (pad_to_mask_clearance 0)
     (pcbplotparams
       (layerselection 0x00010f0_ffffffff)
@@
     (fp_line (start -1.6 0.8) (end -1.6 -0.8) (layer "F.Fab") (width 0.1))
     (fp_line (start 1.6 -0.8) (end 1.6 0.8) (layer "F.Fab") (width 0.1))
-    (pad "1" smd roundrect locked (at -1.475 0) (size 1.15 1.8) (layers "F.Cu" "F.Paste" "F.Mask") (roundrect_rratio 0.217391)
+    (pad "1" smd roundrect locked (at -1.475 0) (size 1.15 1.8) (layers "F.Cu" "F.Paste" "F.Mask") (roundrect_rratio 0.2173913043)
       (net 5 "/VBAT") (pintype "passive"))
-    (pad "2" smd roundrect locked (at 1.475 0) (size 1.15 1.8) (layers "F.Cu" "F.Paste" "F.Mask") (roundrect_rratio 0.217391)
+    (pad "2" smd roundrect locked (at 1.475 0) (size 1.15 1.8) (layers "F.Cu" "F.Paste" "F.Mask") (roundrect_rratio 0.2173913043)
       (net 4 "GND") (pintype "passive"))
     (model "${KISYS3DMOD}/Capacitor_SMD.3dshapes/C_1206_3216Metric.wrl"
@@
     (fp_line (start -3 1) (end 3 1) (layer "F.Fab") (width 0.1))
     (fp_line (start -2.5 -1) (end -3 -0.5) (layer "F.Fab") (width 0.1))
-    (pad "1" smd roundrect locked (at -2.85 0 180) (size 1.2 2.2) (layers "F.Cu" "F.Paste" "F.Mask") (roundrect_rratio 0.208333)
+    (pad "1" smd roundrect locked (at -2.85 0 180) (size 1.2 2.2) (layers "F.Cu" "F.Paste" "F.Mask") (roundrect_rratio 0.2083333333)
       (net 14 "Net-(AE1-Pad1)") (pinfunction "FEED") (pintype "input"))
-    (pad "2" smd roundrect locked (at 2.85 0 180) (size 1.2 2.2) (layers "F.Cu" "F.Paste" "F.Mask") (roundrect_rratio 0.208333)
+    (pad "2" smd roundrect locked (at 2.85 0 180) (size 1.2 2.2) (layers "F.Cu" "F.Paste" "F.Mask") (roundrect_rratio 0.2083333333)
       (net 20 "unconnected-(AE1-Pad2)") (pinfunction "PCB_Trace") (pintype "passive"))
     (model "${KICAD6_3DMODEL_DIR}/RF_Antenna.3dshapes/Johanson_2450AT43F0100.wrl"
@@
     (fp_line (start 1 0.45) (end -1 0.45) (layer "F.Fab") (width 0.1))
     (fp_line (start -1 0.45) (end -1 -0.45) (layer "F.Fab") (width 0.1))
-    (pad "1" smd roundrect locked (at -1.15 0 90) (size 1.05 1.2) (layers "F.Cu" "F.Paste" "F.Mask") (roundrect_rratio 0.238095)
+    (pad "1" smd roundrect locked (at -1.15 0 90) (size 1.05 1.2) (layers "F.Cu" "F.Paste" "F.Mask") (roundrect_rratio 0.2380952381)
       (net 21 "Net-(C3-Pad1)") (pinfunction "1") (pintype "passive"))
-    (pad "2" smd roundrect locked (at 1.15 0 90) (size 1.05 1.2) (layers "F.Cu" "F.Paste" "F.Mask") (roundrect_rratio 0.238095)
+    (pad "2" smd roundrect locked (at 1.15 0 90) (size 1.05 1.2) (layers "F.Cu" "F.Paste" "F.Mask") (roundrect_rratio 0.2380952381)
       (net 14 "Net-(AE1-Pad1)") (pinfunction "2") (pintype "passive"))
     (model "${KICAD6_3DMODEL_DIR}/Inductor_SMD.3dshapes/L_0805_2012Metric.wrl"
@@
     (fp_line (start -1.6 0.8) (end -1.6 -0.8) (layer "F.Fab") (width 0.1))
     (fp_line (start -1.6 -0.8) (end 1.6 -0.8) (layer "F.Fab") (width 0.1))
-    (pad "1" smd roundrect locked (at -1.475 0 90) (size 1.15 1.8) (layers "F.Cu" "F.Paste" "F.Mask") (roundrect_rratio 0.217391)
+    (pad "1" smd roundrect locked (at -1.475 0 90) (size 1.15 1.8) (layers "F.Cu" "F.Paste" "F.Mask") (roundrect_rratio 0.2173913043)
       (net 5 "/VBAT") (pintype "passive"))
-    (pad "2" smd roundrect locked (at 1.475 0 90) (size 1.15 1.8) (layers "F.Cu" "F.Paste" "F.Mask") (roundrect_rratio 0.217391)
+    (pad "2" smd roundrect locked (at 1.475 0 90) (size 1.15 1.8) (layers "F.Cu" "F.Paste" "F.Mask") (roundrect_rratio 0.2173913043)
       (net 4 "GND") (pintype "passive"))
     (model "${KISYS3DMOD}/Capacitor_SMD.3dshapes/C_1206_3216Metric.wrl"
@@
     (pts (xy 94.3 83.5) (xy 61.7 83.5))
     (height 3.5)
-    (gr_text "1283.4646 mils" (at 78 78.85) (layer "Eco1.User")
-      (effects (font (size 1 1) (thickness 0.15)))
-    )
+    (gr_text "32.6000 mm" (at 78 78.85) (layer "Eco1.User")
+      (effects (font (size 1 1) (thickness 0.15)))
+    )

Commit message: Started work on a Rev3
Parts:
- removed C2: 0.1u, Capacitor_SMD:C_0603_1608Metric
- removed U2: LIS2DTW12TR, Package_LGA:LGA-12_2x2mm_P0.5mm
- added Y1: 32.768khz, Crystal:Crystal_SMD_3215-2Pin_3.2x1.5mm, F.Cu at (101.7, 86.3)
- C14: value 1uF -> 44nF
- C15: value 1uF -> 470pF
- R13: value R -> 412
- U1: value RV-3028-C7 -> MCP7940N-xMS; footprint open-Smartwatch:RTC_SMD_MicroCrystal_C7_1.5x3.2mm -> Package_SO:MSOP-8_3x3mm_P0.65mm
- moved U1 17.9 mm to (95.5, 86.9), turned to 0 degrees
- moved J1 3.67 mm to (65.9, 101.6)
Connections:
- U1 pad 1: unconnected-(U1-Pad1) -> Net-(U1-Pad1)
- U1 pad 2: /RTC_INT -> Net-(U1-Pad2)
- U1 pad 3: /SCL -> +3V3
- U1 pad 4: /SDA -> GND
- U1 pad 5: GND -> /SDA
- U1 pad 6: +3V3 -> /SCL
- U1 pad 7: +3V3 -> /RTC_INT
- U1 pad 8: unconnected-(U1-Pad8) -> +3V3
Routing:
- net /SDA: track 43.6 -> 28.6 mm
- net /RTC_INT: track 13.7 -> 1.35 mm, vias 2 -> 1
- net /MOSI: track 11.3 -> 1.96 mm
- net /TFT_DC: track 13.5 -> 4.64 mm
- net +3V3: track 97.2 -> 88.5 mm, vias 6 -> 5
- net /3V3_2: track 19.5 -> 10.8 mm, vias 1 -> 0
- net /TFT_CS: track 11.0 -> 3.04 mm
- net /SCK: track 16.9 -> 9.07 mm
- net /TFT_RST: track 20.4 -> 13.3 mm
- net Net-(C23-Pad1): track 12.0 -> 5.91 mm, vias 2 -> 1
- net /SCL: track 42.0 -> 37.0 mm
- net GND: track 16.0 -> 11.4 mm, vias 34 -> 32
- net /LEDK: track 3.63 -> 1.24 mm, vias 1 -> 0
- net /FLASH: vias 2 -> 1
